File: subsystems/mikrobus/mikrobus.kicad_sch (KiCad schematic)
At the start: 3 parts, among them J5 MIKROE-4247

Commit message: Mikrobus bug fix. fp and sym lib table address changes
Parts:
- J5: footprint Com_L432KC_footprint:MIKROE4247 -> User:MIKROE4247; symbol Com_L432KC_symbols:MIKROE-4247 -> Mikrobus:MIKROE-4247
Changed lines of the file:
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@@
 	)
 	(symbol
-		(lib_id "Com_L432KC_symbols:MIKROE-4247")
+		(lib_id "Mikrobus:MIKROE-4247")
 		(at 144.78 99.06 180)
 		(unit 1)
@@
 			)
 		)
-		(property "Footprint" "Com_L432KC_footprint:MIKROE4247"
+		(property "Footprint" "User:MIKROE4247"
 			(at 118.11 4.14 0)
 			(effects
