File: subsystems/mikrobus/mikrobus.kicad_pcb (KiCad board)
At the start: 2 copper layers, 3 parts, among them J1 MIKROE-4247

Commit message: changes to readme. Test list
Parts:
- J1: footprint User:MIKROE4247 -> Mikrobus:MIKROE4247
Changed lines of the file:
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@@
 		)
 	)
-	(footprint "User:MIKROE4247"
+	(footprint "Mikrobus:MIKROE4247"
 		(layer "F.Cu")
 		(at 110.22 83.5)
