File: subsystems/can_buffer/can_buffer.kicad_pcb (KiCad board)
At the start: 2 copper layers, 7 parts

Commit message: Pcb (#25)
* Basic pcb inclusion.

* Group pcb items per template.

* piece of software used to move pcb whole sections and get their limits based on F_crtyrd

---------

Co-authored-by: GivaldoEc <givaldo.t.santos@gmail.com>
Parts:
- moved C2 37.8 mm to (136.8, 71.2)
- moved C1 37.8 mm to (136.8, 68.2)
- moved R1 37.1 mm to (134.0, 62.8)
- moved R2 37.1 mm to (134.0, 65.0)
- moved CR1 31.9 mm to (141.0, 62.0)
- moved JP1 28.8 mm to (146.6, 56.4), turned to 90 degrees
- moved R3 22.0 mm to (147.5, 59.9), turned to 180 degrees
Routing:
- net GND: track 12.6 -> 0.00 mm
- net Net-(CR1-VS): track 9.78 -> 12.2 mm
- net Net-(CR1-ASC): track 9.01 -> 6.56 mm
